Commit message: CAD and inertial

File: description/robot.urdf (robot description, URDF)
Before this commit: robot robot, 5 links, 4 joints
Links:
- link forearm: mass 0 -> 722.16061394
- link shoulder: mass 0 -> 445.83607510
- link upperarm: mass 0 -> 1897.69177373

Commit message: Joint offsets

File: description/robot.urdf (robot description, URDF)
Before this commit: robot robot, 5 links, 4 joints
Joints:
- joint forearm: origin xyz=0 0 0 rpy=0 0 0 -> xyz=3.5 0 0 rpy=0 0 0
- joint shoulder: origin xyz=0 0 0 rpy=0 0 0 -> xyz=0 0 1 rpy=1.5708 0 0
- joint wrist: origin xyz=0 0.0 0.0 rpy=0 0 0 -> xyz=3.5 0.0 0.0 rpy=0 0 0

Commit message: Adjust geometry and limits

File: description/robot.urdf (robot description, URDF)
Before this commit: robot robot, 5 links, 4 joints
Joints:
- joint forearm: axis 0 1 0 -> 0 0 1; limit lower=-1.5708 upper=1.5708 effort=100 velocity=1.0 -> lower=-1.5708 upper=0 effort=100 velocity=1.0
- joint upperarm: axis 0 1 0 -> 0 0 1; limit lower=-1.5708 upper=1.5708 effort=100 velocity=1.0 -> lower=-0.8417 upper=1.5708 effort=100 velocity=1.0

Commit message: Ensure joint names are unique

File: description/robot.urdf (robot description, URDF)
Before this commit: robot robot, 5 links, 4 joints
Joints:
- removed joint forearm
- removed joint shoulder
- removed joint upperarm
- added joint forearm_joint: type revolute, parent upperarm, child forearm, origin xyz=3.5 0 0 rpy=0 0 0, axis 0 0 1, limit lower=-1.5708 upper=0 effort=100 velocity=1.0
- added joint shoulder_joint: type revolute, parent world, child shoulder, origin xyz=0 0 1 rpy=1.5708 0 0, axis 0 1 0, limit lower=-1.5708 upper=1.5708 effort=100 velocity=1.0
- added joint upperarm_joint: type revolute, parent shoulder, child upperarm, origin xyz=0 0 0 rpy=0 0 0, axis 0 0 1, limit lower=-0.8417 upper=1.5708 effort=100 velocity=1.0

Commit message: Get basic velocity control working

File: description/robot.urdf (robot description, URDF)
Before this commit: robot robot, 5 links, 4 joints
Joints:
- joint forearm_joint: limit lower=-1.5708 upper=0 effort=100 velocity=1.0 -> lower=-1.5708 upper=0 effort=100000 velocity=1.0
- joint shoulder_joint: limit lower=-1.5708 upper=1.5708 effort=100 velocity=1.0 -> lower=-1.5708 upper=1.5708 effort=100000 velocity=1.0
- joint upperarm_joint: limit lower=-0.8417 upper=1.5708 effort=100 velocity=1.0 -> lower=-0.8417 upper=1.5708 effort=100000 velocity=1.0

Commit message: Add gripper joints and links

File: description/robot.urdf (robot description, URDF)
Before this commit: robot robot, 5 links, 4 joints
Links:
- added link gripper_bottom, mass 0; collision mesh filename=package://basic_velocity_control/description/models/gripper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; visual mesh filename=package://basic_velocity_control/description/models/gripper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
- added link gripper_top, mass 0; collision mesh filename=package://basic_velocity_control/description/models/gripper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; visual mesh filename=package://basic_velocity_control/description/models/gripper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
Joints:
- added joint gripper_bottom_joint: type prismatic, parent forearm, origin xyz=3.5 0.0 0.0 rpy=0 0 0, axis 0 0 1, limit lower=0.01 upper=0 effort=100000 velocity=1.0
- added joint gripper_top_joint: type prismatic, parent forearm, origin xyz=3.5 0.0 0.0 rpy=0 0 0, axis 0 0 1, limit lower=-0.01 upper=0 effort=100000 velocity=1.0

Commit message: Add gripper

File: description/robot.urdf (robot description, URDF)
Before this commit: robot robot, 7 links, 6 joints
Joints:
- joint gripper_bottom_joint: child (none) -> gripper_bottom; limit lower=0.01 upper=0 effort=100000 velocity=1.0 -> lower=0 upper=0.0688 effort=100000 velocity=1.0; origin xyz=3.5 0.0 0.0 rpy=0 0 0 -> xyz=3.65 0.0 0.0 rpy=1.5708 0 0
- joint gripper_top_joint: child (none) -> gripper_top; limit lower=-0.01 upper=0 effort=100000 velocity=1.0 -> lower=-0.0688 upper=0 effort=100000 velocity=1.0; origin xyz=3.5 0.0 0.0 rpy=0 0 0 -> xyz=3.65 0.0 0.0 rpy=1.5708 0 0

Commit message: Re-generate moveit config

File: description/robot.urdf (robot description, URDF)
Before this commit: robot robot, 7 links, 6 joints
Joints:
- joint gripper_bottom_joint: origin xyz=3.65 0.0 0.0 rpy=1.5708 0 0 -> xyz=0.15 0.0 0.0 rpy=1.5708 0 0; parent forearm -> tool
- joint gripper_top_joint: origin xyz=3.65 0.0 0.0 rpy=1.5708 0 0 -> xyz=0.15 0.0 0.0 rpy=1.5708 0 0; parent forearm -> tool

Commit message: Add dummy physical properties for gripper

File: description/robot.urdf (robot description, URDF)
Before this commit: robot robot, 7 links, 6 joints
Links:
- link gripper_bottom: mass 0 -> 1.0
- link gripper_top: mass 0 -> 1.0
- link tool: mass 0 -> 1.0; geometry collision sphere radius=0.1; visual sphere radius=0.05

Commit message: Make gripper joints mimics

File: description/robot.urdf (robot description, URDF)
Before this commit: robot robot, 7 links, 6 joints
Joints:
- removed joint gripper_bottom_joint
- removed joint gripper_top_joint
- added joint gripper: type prismatic, parent tool, origin xyz=0.15 0.0 0.0 rpy=1.5708 0 0, limit lower=0 upper=0.0688 effort=100000 velocity=1.0, mimic joint=gripper_top_mimic multiplier=-1.0 offset=0.0
- added joint gripper_bottom_mimic: type prismatic, parent tool, child gripper_bottom, origin xyz=0.15 0.0 0.0 rpy=1.5708 0 0, axis 0 0 1, limit lower=0 upper=0.0688 effort=100000 velocity=1.0
- added joint gripper_top_mimic: type prismatic, parent tool, child gripper_top, origin xyz=0.15 0.0 0.0 rpy=1.5708 0 0, axis 0 0 1, limit lower=-0.0688 upper=0 effort=100000 velocity=1.0

Commit message: Single gripper

File: description/robot.urdf (robot description, URDF)
Before this commit: robot robot, 7 links, 7 joints
Links:
- added link dummy
Joints:
- joint gripper: child (none) -> dummy

Commit message: Wrong mimic direction

File: description/robot.urdf (robot description, URDF)
Before this commit: robot robot, 8 links, 7 joints
Joints:
- joint gripper: mimic joint=gripper_top_mimic multiplier=-1.0 offset=0.0 -> (none)
- joint gripper_bottom_mimic: mimic (none) -> joint=gripper multiplier=1.0 offset=0.0
- joint gripper_top_mimic: mimic (none) -> joint=gripper multiplier=-1.0 offset=0.0

Commit message: Add physical properties for dummy so Gazebo can load it

File: description/robot.urdf (robot description, URDF)
Before this commit: robot robot, 8 links, 7 joints
Links:
- removed link world
- link dummy: mass None -> 1.0; geometry collision sphere radius=0.1; visual sphere radius=0.05

Commit message: Put world link back in

File: description/robot.urdf (robot description, URDF)
Before this commit: robot robot, 7 links, 7 joints
Links:
- added link world

Commit message: Re-export models and update urdf

File: description/robot.urdf (robot description, URDF)
Before this commit: robot robot, 8 links, 7 joints
Links:
- removed link dummy
- removed link gripper_bottom
- removed link gripper_top
- removed link shoulder
- added link base, mass 27.291; collision mesh filename=package://basic_velocity_control/description/models/base.stl; visual mesh filename=package://basic_velocity_control/description/models/base.stl
- added link finger1, mass 1.08815625; collision mesh filename=package://basic_velocity_control/description/models/finger1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; visual mesh filename=package://basic_velocity_control/description/models/finger1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
- added link finger2, mass 1.08815625; collision mesh filename=package://basic_velocity_control/description/models/finger2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; visual mesh filename=package://basic_velocity_control/description/models/finger2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
- added link hand, mass 10.32823427; collision mesh filename=package://basic_velocity_control/description/models/hand.stl; visual mesh filename=package://basic_velocity_control/description/models/hand.stl
- link forearm: mass 722.16061394 -> 36.13666037
- link tool: mass 1.0 -> 0.00000001; geometry collision sphere radius=0.5; visual sphere radius=0.5
Joints:
- removed joint forearm_joint
- removed joint shoulder_joint
- removed joint upperarm_joint
- added joint base: type revolute, parent world, child shoulder, origin xyz=0 0 0 rpy=0 0 0, axis 0 0 1, limit lower=-1.5708 upper=1.5708 effort=100000 velocity=1.0
- added joint elbow: type revolute, parent upperarm, child forearm, origin xyz=0.7 0 0 rpy=0 0 0, axis 0 1 1, limit lower=-1.5708 upper=0 effort=100000 velocity=1.0
- added joint shoulder: type revolute, parent shoulder, child upperarm, origin xyz=0 0 0.670 rpy=0 0 0, axis 0 1 0, limit lower=-0.8417 upper=1.5708 effort=100000 velocity=1.0
- joint gripper: axis (none) -> 0 1 0; child dummy -> tool; limit lower=0 upper=0.0688 effort=100000 velocity=1.0 -> lower=0 upper=0.07 effort=100000 velocity=1.0; origin xyz=0.15 0.0 0.0 rpy=1.5708 0 0 -> xyz=0.0 0.0 0.0 rpy=0 0 0; parent tool -> hand
- joint gripper_bottom_mimic: axis 0 0 1 -> 0 1 0; child gripper_bottom -> finger1; limit lower=0 upper=0.0688 effort=100000 velocity=1.0 -> lower=0 upper=0.07 effort=100000 velocity=1.0; origin xyz=0.15 0.0 0.0 rpy=1.5708 0 0 -> xyz=0.0 0.0 0.0 rpy=0 0 0; parent tool -> hand
- joint gripper_top_mimic: axis 0 0 1 -> 0 1 0; child gripper_top -> finger2; limit lower=-0.0688 upper=0 effort=100000 velocity=1.0 -> lower=-0.07 upper=0 effort=100000 velocity=1.0; origin xyz=0.15 0.0 0.0 rpy=1.5708 0 0 -> xyz=0.0 0.0 0.0 rpy=0 0 0; parent tool -> hand
- joint wrist: axis (none) -> 1 0 0; limit (none) -> lower=-1.5708 upper=1.5708 effort=100000 velocity=1.0; origin xyz=3.5 0.0 0.0 rpy=0 0 0 -> xyz=0.7 0.05 0.0 rpy=0 0 0

Commit message: Fix issues in URDF

File: description/robot.urdf (robot description, URDF)
Before this commit: robot robot, 8 links, 7 joints
Links:
- removed link tool
- added link dummy, mass 1.08815625; collision sphere radius=0.01; visual sphere radius=0.01
Joints:
- removed joint base
- removed joint elbow
- removed joint gripper
- removed joint gripper_bottom_mimic
- removed joint gripper_top_mimic
- removed joint shoulder
- removed joint wrist
- added joint base_joint: type revolute, parent world, child base, origin xyz=0 0 0 rpy=0 0 0, axis 0 0 1, limit lower=-1.5708 upper=1.5708 effort=100000 velocity=1.0
- added joint elbow_joint: type revolute, parent upperarm, child forearm, origin xyz=0.7 0 0 rpy=0 0 0, axis 0 1 0, limit lower=0 upper=1.5708 effort=100000 velocity=1.0
- added joint finger1_joint: type prismatic, parent hand, child finger1, origin xyz=0 0 0 rpy=0 0 0, axis 0 1 0, limit lower=0 upper=0.07 effort=100000 velocity=1.0, mimic joint=finger_joint multiplier=1.0 offset=0.0
- added joint finger2_joint: type prismatic, parent hand, child finger2, origin xyz=0 0 0 rpy=0 0 0, axis 0 1 0, limit lower=-0.07 upper=0 effort=100000 velocity=1.0, mimic joint=finger_joint multiplier=-1.0 offset=0.0
- added joint finger_joint: type prismatic, parent hand, child dummy, origin xyz=0 0 0 rpy=0 0 0, axis 0 1 0, limit lower=0 upper=0.07 effort=100000 velocity=1.0
- added joint shoulder_joint: type revolute, parent base, child upperarm, origin xyz=0 0 0.670 rpy=0 0 0, axis 0 1 0, limit lower=-0.8417 upper=1.5708 effort=100000 velocity=1.0
- added joint wrist_joint: type revolute, parent forearm, child hand, origin xyz=0.7 0.05 0.0 rpy=0 0 0, axis 1 0 0, limit lower=-1.5708 upper=1.5708 effort=100000 velocity=1.0
